File: LineFollower/TCRT1010_VIS.pac.sch (EAGLE design)
At the start: 10 parts, among them U1 TCRT5000, U2 LM358DR

Commit message: 5 channel module
Parts:
- added D3, D4, D5, D6: LED5MM, MIA_LIBRARY-2-2-2:LED5MM
- added JP2: (no value), MIA_LIBRARY-2-2-2:PINHD-1X7
- added R10, R14, R18, R6: (no value), MIA_LIBRARY-2-2-2:TRIM_EU-CA6V
- added R11, R15, R19, R7: 100, MIA_LIBRARY-2-2-2:RES-7
- added R12, R16, R20, R8: 10k, MIA_LIBRARY-2-2-2:RES-7
- added R13, R17, R21, R9: 330, MIA_LIBRARY-2-2-2:RES-7
- added U3, U4, U6, U7: TCRT5000, TCRT5000:TCRT5000
- added U5, U9: LM358, MIA_LIBRARY-2-2-2:LM358
- D1, D2: value (none) -> LED5MM; device 52101-101-REV-A_v16:LED_LEDCHIP-LED0603MP -> MIA_LIBRARY-2-2-2:LED5MM
- JP1: device MIA_LIBRARY-2-2-2:PINHD-1X4 -> MIA_LIBRARY-2-2-2:PINHD-1X7
- R2: device rcl:R-US_R0805 -> MIA_LIBRARY-2-2-2:RES-7
- R3, R4, R5: device rcl:R-US_R0603 -> MIA_LIBRARY-2-2-2:RES-7
- U2: value LM358DR -> LM358; device IC:LM358DR -> MIA_LIBRARY-2-2-2:LM358
Connections:
- new net D1: D3.A, JP2.4, R9.1
- new net D2: D4.A, JP2.5, R13.1
- new net D3: D5.A, JP2.6, R17.1
- new net D4: D6.A, JP2.7, R21.1
- new net IN3+: R10.S, U2G1.+IN
- new net IN3-: JP1.5, R12.2, U2G1.-IN, U4.E
- new net IN4+: R14.S, U2G2.+IN
- new net IN4-: JP1.6, R16.2, U2G2.-IN, U6.E
- new net IN5+: U5G1.+IN
- new net IN5-: U5G1.-IN
- new net IN6+: R18.S, U5G2.+IN
- new net IN6-: JP1.7, R20.2, U5G2.-IN, U7.E
- new net N$3: R7.2, U3.CATH
- new net N$4: R11.2, U4.CATH
- new net N$5: R15.2, U6.CATH
- new net N$6: R19.2, U7.CATH
- new net OUT3: R13.2, U2G1.OUT
- new net OUT4: R17.2, U2G2.OUT
- new net OUT5: U5G1.OUT
- new net OUT6: R21.2, U5G2.OUT
- net D0: now also JP2.3; no longer JP1.4
- net GND: now also D3.C, D4.C, D5.C, D6.C, JP2.2, R10.A, R11.1, R12.1, R14.A, R15.1, R16.1, R18.A, R19.1, R20.1, R6.A, R7.1, R8.1, U2G3.P$V-, U5G3.P$V-, U9G3.P$V-; no longer U2.V-
- net IN1+: now also U9G1.+IN; no longer U2.IN1+
- net IN1-: now also U9G1.-IN; no longer U2.IN1-
- net IN2+: now also R6.S, U9G2.+IN; no longer U2.IN2+
- net IN2-: now also JP1.4, R8.2, U3.E, U9G2.-IN; no longer U2.IN2-
- net OUT1: now also U9G1.OUT; no longer U2.OUT1
- net OUT2: now also R9.2, U9G2.OUT; no longer U2.OUT2
- net VCC: now also JP2.1, R10.E, R14.E, R18.E, R6.E, U2G3.P$V+, U3.A, U3.COLL, U4.A, U4.COLL, U5G3.P$V+, U6.A, U6.COLL, U7.A, U7.COLL, U9G3.P$V+; no longer U2.V+
Other:
- moved on the sheet: D1, D2, R1, R2, R3, R4, R5, U1
